File: digitalOut.kicad_sch (KiCad schematic)
At the start: 4 parts, among them J18 Conn_02x04_Odd_Even, J22 AudioJack2_SwitchT, U4 74AHCT1G126GV

Commit message: Switched to two layers
Connections:
- net +12V: no longer names the net of J18.1 (Pin_1)
- net -12V: no longer names the net of J18.7 (Pin_7)
Changed lines of the file:
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@@
   (junction (at 124.46 63.5) (diameter 0) (color 0 0 0 0)
-  )
-  (wire (pts (xy 71.12 59.69) (xy 71.12 68.58))
-    (stroke (width 0) (type default) (color 0 0 0 0))
   )
   (wire (pts (xy 87.63 76.2) (xy 89.535 76.2))
@@
     (stroke (width 0) (type default) (color 0 0 0 0))
   )
-  (wire (pts (xy 74.93 76.2) (xy 73.025 76.2))
-    (stroke (width 0) (type default) (color 0 0 0 0))
-  )
   (wire (pts (xy 74.93 73.66) (xy 60.96 73.66))
-    (stroke (width 0) (type default) (color 0 0 0 0))
-  )
-  (wire (pts (xy 73.025 76.2) (xy 73.025 78.74))
     (stroke (width 0) (type default) (color 0 0 0 0))
   )
@@
   )
   (wire (pts (xy 109.22 68.58) (xy 115.57 68.58))
-    (stroke (width 0) (type default) (color 0 0 0 0))
-  )
-  (wire (pts (xy 74.93 68.58) (xy 71.12 68.58))
     (stroke (width 0) (type default) (color 0 0 0 0))
   )
@@
     (pin "1")
   )
-  (symbol (lib_id "power:-12V") (at 73.025 78.74 0) (mirror x) (unit 1)
-    (in_bom yes) (on_board yes) (fields_autoplaced)
-    (property "Reference" "#PWR0154" (id 0) (at 73.025 81.28 0)
-      (effects (font (size 1.27 1.27)) hide)
-    )
-    (property "Value" "-12V" (id 1) (at 73.025 83.82 0))
-    (property "Footprint" "" (id 2) (at 73.025 78.74 0)
-      (effects (font (size 1.27 1.27)) hide)
-    )
-    (property "Datasheet" "" (id 3) (at 73.025 78.74 0)
-      (effects (font (size 1.27 1.27)) hide)
-    )
-    (pin "1")
-  )
   (symbol (lib_id "power:GND") (at 89.535 79.375 0) (mirror y) (unit 1)
     (in_bom yes) (on_board yes) (fields_autoplaced)
@@
       (effects (font (size 1.27 1.27)) hide)
     )
-    (pin "1")
-  )
-  (symbol (lib_id "power:+12V") (at 71.12 59.69 0) (mirror y) (unit 1)
-    (in_bom yes) (on_board yes) (fields_autoplaced)
-    (property "Reference" "#PWR0153" (id 0) (at 71.12 63.5 0)
-      (effects (font (size 1.27 1.27)) hide)
-    )
-    (property "Value" "+12V" (id 1) (at 71.12 54.61 0))
-    (property "Footprint" "" (id 2) (at 71.12 59.69 0)
-      (effects (font (size 1.27 1.27)) hide)
-    )
-    (property "Datasheet" "" (id 3) (at 71.12 59.69 0)
-      (effects (font (size 1.27 1.27)) hide)
-    )
