File: vestmannaeyjar.kicad_sch (KiCad schematic)
At the start: 3 parts, among them J37 USB_B, U3 DKM10E-12

Commit message: Switched to two layers
Parts:
- J33: value (none) -> Conn_02x08_Odd_Even; footprint (none) -> Connector_PinHeader_2.54mm:PinHeader_2x08_P2.54mm_Vertical
- U3: value DKM10E-12 -> (none); footprint parts:DKM10 -> (none)
